File: hardware/sdr_analogic/sdr.sch (KiCad schematic (older format))
At the start: 73 parts, among them J1 Conn_01x02, J2 Conn_01x01, U1 LM4562, U2 LM4562, U3 LM4562, U4 TS3A5017, U5 LM4562, U6 LM4562

Commit message: schematic update
Parts:
- added C?: 80-C1206C475K5R, Capacitor_SMD:C_1206_3216Metric_Pad1.42x1.75mm_HandSolder, symbol Device:C_Small
- added C? (x6): 100n, Capacitor_SMD:C_1206_3216Metric_Pad1.42x1.75mm_HandSolder, symbol Device:C_Small
- added R? (x2): 1k, Resistor_SMD:R_1206_3216Metric_Pad1.42x1.75mm_HandSolder, symbol Device:R_Small
- added R? (x2): 100, Resistor_SMD:R_1206_3216Metric_Pad1.42x1.75mm_HandSolder, symbol Device:R_Small
Connections:
- net +12V: now also R?.1
- net AMP_BIAS: now also C?.1, C?.1, C?.1, C?.1, C?.1, C?.1, C?.1, R?.1, R?.2
- net GND: now also C?.2, C?.2, C?.2, C?.2, C?.2, C?.2, C?.2, R?.2
- net at R14.2, U2.6 (-): now also R?.2; no longer R11.1
- net at R15.2, U3.2 (-): now also R?.2; no longer R12.2
- net at R16.2, U3.6 (-): now also R12.2; no longer R12.1
- new net: R11.1, R?.1
- new net: R12.1, R?.1
Other:
- note added: "discrete instrumentation amplifier\nuse precision parts"
- note added: "quadrature mixer and LO\nI2C isolator"
- note removed: "quadrature mixer"
- moved on the sheet: C10, C11, C12, C7, C8, C9, C?, J2, J?, R10, R11, R12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

Commit message: schematic ready for layout
Parts:
- removed C?: 100n, Capacitor_SMD:C_1206_3216Metric_Pad1.42x1.75mm_HandSolder, symbol Device:C_Small
- removed J?: AudioJack3_Ground, symbol Connector:AudioJack3_Ground
- C10, C11, C12, C7, C8, C9: value 1u -> R82DC4100AA60K
- C13: renamed from C?; value 100u -> 1000u/25V; footprint Capacitor_SMD:C_1206_3216Metric -> Capacitor_THT:CP_Radial_D13.0mm_P5.00mm
- C20: renamed from C?; value 100u -> 1000u/10V; footprint Capacitor_SMD:C_1206_3216Metric -> Capacitor_THT:CP_Radial_D10.0mm_P5.00mm
- C3, C4, C5, C6: value R82DC3100AA50J -> ECH-U1C104GX5; footprint Capacitor_THT:C_Rect_L7.2mm_W4.5mm_P5.00mm_FKS2_FKP2_MKS2_MKP2 -> Capacitor_SMD:C_1210_3225Metric_Pad1.42x2.65mm_HandSolder
- FB1, FB2, FB3: renamed from FB?; footprint (none) -> Resistor_SMD:R_1206_3216Metric
- J1: footprint (none) -> Connector_PinSocket_2.54mm:PinSocket_1x02_P2.54mm_Vertical
- J2: footprint (none) -> Connector_PinSocket_2.54mm:PinSocket_1x01_P2.54mm_Vertical
- J3: renamed from J?; footprint (none) -> Connector_PinSocket_2.54mm:PinSocket_1x02_P2.54mm_Vertical
- J4: renamed from J?; footprint (none) -> Connector_PinSocket_2.54mm:PinSocket_1x04_P2.54mm_Vertical
- J6: renamed from J?; footprint (none) -> Connector_PinSocket_2.54mm:PinSocket_1x03_P2.54mm_Vertical
- U1: value LM4562 -> ETC4-1-2TR; footprint (none) -> sdr_analogic:ETC4-1-2TR
- U10, U9: renamed from U?; footprint (none) -> sdr_analogic:LM-NP-1001-B1L
- U2, U3, U6: value LM4562 -> LM4562MAX/NOPB; footprint (none) -> Package_SO:SOIC-8_5.23x5.23mm_P1.27mm
- U4: value TS3A5017 -> TS3A5017DR; footprint (none) -> Package_SO:SOIC-16W_5.3x10.2mm_P1.27mm
- U5: value LM4562 -> Si5351A-B-GT; footprint (none) -> Package_SO:MSOP-10_3x3mm_P0.5mm
- U7: renamed from U?; footprint (none) -> Package_SO:SOIC-8_3.9x4.9mm_P1.27mm
- Y1: renamed from Y?; footprint (none) -> sdr_analogic:XRCGB25M000F1H00R0
- gave numbers to parts that had none: 26

Commit message: redesign projec for https://github.com/ArjanteMarvelde/uSDR-pico
Parts:
- removed C1: 1n, Capacitor_SMD:C_1206_3216Metric, symbol Device:C_Small
- removed C10, C11, C12, C7, C8, C9: R82DC4100AA60K, Capacitor_SMD:C_1206_3216Metric, symbol Device:C_Small
- removed C13: 1000u/25V, Capacitor_THT:CP_Radial_D13.0mm_P5.00mm, symbol Device:C_Small
- removed C14, C17, C18, C19, C21, C22, C24, C26, C29, C30, C31, C32, C33, C34: 100n, Capacitor_SMD:C_1206_3216Metric_Pad1.42x1.75mm_HandSolder, symbol Device:C_Small
- removed C15, C23, C25, C27, C28: 80-C1206C475K5R, Capacitor_SMD:C_1206_3216Metric_Pad1.42x1.75mm_HandSolder, symbol Device:C_Small
- removed C2: 100n, Capacitor_SMD:C_1206_3216Metric, symbol Device:C_Small
- removed C20: 1000u/10V, Capacitor_THT:CP_Radial_D10.0mm_P5.00mm, symbol Device:C_Small
- removed C3, C4, C5, C6: ECH-U1C104GX5, Capacitor_SMD:C_1210_3225Metric_Pad1.42x2.65mm_HandSolder, symbol Device:C_Small
- removed FB1, FB2, FB3: HZ1206C202R-10, Resistor_SMD:R_1206_3216Metric, symbol Device:Ferrite_Bead_Small
- removed J1, J3: Conn_01x02, Connector_PinSocket_2.54mm:PinSocket_1x02_P2.54mm_Vertical, symbol Connector_Generic:Conn_01x02
- removed J2: Conn_01x01, Connector_PinSocket_2.54mm:PinSocket_1x01_P2.54mm_Vertical, symbol Connector_Generic:Conn_01x01
- removed J4: Conn_01x04, Connector_PinSocket_2.54mm:PinSocket_1x04_P2.54mm_Vertical, symbol Connector_Generic:Conn_01x04
- removed J6: Conn_01x03, Connector_PinSocket_2.54mm:PinSocket_1x03_P2.54mm_Vertical, symbol Connector_Generic:Conn_01x03
- removed R1, R2, R3, R4, R5, R6: 1K, Resistor_SMD:R_1206_3216Metric_Pad1.42x1.75mm_HandSolder, symbol Device:R_Small
- removed R10, R13, R15, R17, R18, R19, R20, R21, R22, R23, R24, R7, R8, R9: 10K, Resistor_SMD:R_1206_3216Metric_Pad1.42x1.75mm_HandSolder, symbol Device:R_Small
- removed R11, R12, R27, R28: 100, Resistor_SMD:R_1206_3216Metric_Pad1.42x1.75mm_HandSolder, symbol Device:R_Small
- removed R14, R16: 10k, Resistor_SMD:R_1206_3216Metric_Pad1.42x1.75mm_HandSolder, symbol Device:R_Small
- removed R25, R26: 4.7k, Resistor_SMD:R_1206_3216Metric_Pad1.42x1.75mm_HandSolder, symbol Device:R_Small
- removed R29, R30: 1k, Resistor_SMD:R_1206_3216Metric_Pad1.42x1.75mm_HandSolder, symbol Device:R_Small
- removed U1: ETC4-1-2TR, sdr_analogic:ETC4-1-2TR, symbol sdr:ETC4-1-2TR
- removed U10, U9: LM-NP-1001-B1L, sdr_analogic:LM-NP-1001-B1L, symbol sdr:LM-NP-1001-B1L
- removed U2, U3, U6: LM4562MAX/NOPB, Package_SO:SOIC-8_5.23x5.23mm_P1.27mm, symbol Amplifier_Operational:LM4562
- removed U4: TS3A5017DR, Package_SO:SOIC-16W_5.3x10.2mm_P1.27mm, symbol sdr:TS3A5017
- removed U5: Si5351A-B-GT, Package_SO:MSOP-10_3x3mm_P0.5mm, symbol Oscillator:Si5351A-B-GT
- removed U7: SI8602AC-B-ISR, Package_SO:SOIC-8_3.9x4.9mm_P1.27mm, symbol sdr:SI8602AC-B-ISR
- removed U8: LD1086D2T33TR, Package_TO_SOT_SMD:TO-263-2, symbol Regulator_Linear:LD1086D2T33TR
- removed Y1: XRCGB25M000F1H00R0, sdr_analogic:XRCGB25M000F1H00R0, symbol Device:Crystal_Small
- added J?: Conn_Coaxial, symbol Connector:Conn_Coaxial
- added J? (x2): Conn_01x02, symbol Connector_Generic:Conn_01x02
Connections:
- net GND: now also J?.2 (Ext), J?.2 (Pin_2), J?.2 (Pin_2)
- new net AudioOut/AUDIO_POWER_OUT: J?.1 (Pin_1)
- new net Mixer/RF_IN: J?.1 (In)
- new net Power/VCC: J?.1 (Pin_1)
Other:
- note removed: "discrete instrumentation amplifier\nuse precision parts"
- note removed: "quadrature mixer and LO\nI2C isolator"
